File: Hardware/0. Project/It's Time, Do.sch (EAGLE design)
At the start: 8 parts, among them U5 MCP6024

Commit message: WIP
Parts:
- removed C26: 100nF x 50V, My-RLC:C_0603
- removed R21: 220R (5%), My-RLC:R_0603
- removed R27: 1k4 (0.5%), My-RLC:R_0603
- removed R32, R33: 100k (0.5%), My-RLC:R_0603
- removed U5: MCP6024, MCP6024:MCP6024
Connections:
- net ADC_VOLTAGE_L1 renamed N$1
- removed net 3.3V: C26.2, U5G$1.V+
- removed net AGND-V: R27.2, R32.2
- removed net N$15: R23.2, R33.1, U5A.OUT
- removed net N$30: R32.1, R33.2, U5A.-IN
- removed net N$31: R21.2, R27.1
- removed net N$32: R21.1, U5A.+IN
- net 0V: no longer C26.1, U5G$1.V-
Other:
- note removed: "Vp-max 1,50V"
