File: Hardware/0. Project/It-s Time, Do.brd (EAGLE design)
At the start: 50 x 50 mm, 66 parts, among them CN1 USB 3.2 Gen 2 Type C Receptac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, CN2 3P-MINI-FIT-JR, CN3 2P-MINI-FIT-JR, CN4 JTAG, CN5 CELL-CONNECTOR, CN6 CR-1220, Q1 BC817, Q2 NPN-BC817, Q3 NPN-BC817, Q4 P-FET-ENHANCEMENT-SI2369BDS, U1 CP2102N, U2 LMV321, U3 MCP73831, U4 TLV75530PDBVR, U5 DS3231-SO16

Commit message: PCB v1.0 release
Parts:
- removed C21: 100nF, My-RLC:C0603
- removed DS1: 0.96" active Area / 128x64 pixels, My-Displays:OLED-RAW-0.96"
- removed R20: 100R (5%), My-RLC:R0603
- removed R21, R22: 4k7 (5%), My-RLC:R0603
- removed R23: 390k (1%), My-RLC:R0603
- removed R24, R25: 10k (5%), My-RLC:R0603
- C1: value 100nF -> 4.7nF x 100V
- C10: value 100nF -> 100nF x 50V
- C11: value 1nF -> 100nF
- C12: value 100uF x 10V -> 100nF; device My-RLC:PTH-5MM -> My-RLC:C0603
- C15: value 100nF -> 10nF
- C16: value 100nF -> 100uF x 10V; device My-RLC:C0603 -> My-RLC:PTH-5MM
- C17: value 10uF -> 10uF x 10V; device My-RLC:C0603 -> My-RLC:C1206_POL
- C18, C9: value 10uF -> 100nF x 50V
- C19: value 10uF -> 22uF x 6.3V; device My-RLC:C0603 -> My-RLC:C1206_POL
- C2: value 4.7nF -> 100nF x 50V
- C20: value 1uF -> 100nF x 50V
- C3: value 100nF -> 10uF x 6.3V
- C4: value 10uF -> 10uF x10V
- C5: value 100nF -> 1nF x 50V
- C6: value 10nF -> 10uF x 6.3V
- C7: value 10uF -> 1uF x 6.3V
- C8: value 1nF -> 1nF x 50V
- CN1: value USB 3.2 Gen 2 Type C Receptacle -> USB Type C Receptacle; device My-Connectors:USB-C-24P -> My-Connectors:USB-C-16P-2LAYER-PADS
- CN2: value 3P-MINI-FIT-JR -> OLED-MODULE-I2C-SOCKET; device My-Connectors:MINI-FIT-JR-3P -> My-Displays:PIN_HEADER_1X4_FEMALE
- CN4: value JTAG -> CR1220; device My-Connectors:JTAG-ARM-10P -> My-Battery:CR1220/1225_HOLDER2
- CN5: value CELL-CONNECTOR -> BATTERY; device My-Battery:JST-PH2 -> My-Battery:JST-PH-2P-H
- CN6: value CR-1220 -> 3P-MINI-FIT-JR; device My-Battery:CR1220/1225_HOLDER -> My-Connectors:MINI-FIT-JR-3P
- Q1: value BC817 -> NPN-BC817
- Q3: value NPN-BC817 -> BC817
- R1: value 22R (5%) -> 1M (5%)
- R10: value 10k (5%) -> 22K (5%)
- R11, R7: value 4k7 (5%) -> 10k (5%)
- R12: value 10k (5%) -> 47R (5%)
- R13: value 47R (5%) -> 4k7 (5%)
- R14: value 22K (5%) -> 10k (5%)
- R15: value 24k (5%) -> 100R (5%)
- R16: value 47k (5%) -> 24k (5%)
- R17: value 10k (5%) -> 47k (5%)
- R2: value 22R (5%) -> 4k7 (5%)
- R4: value 1M (5%) -> 5k1 (1%)
- R6: value 10k (5%) -> 4k7 (5%)
- R9: value 5k1 (5%) -> 4k7 (5%)
- SOC1: value ESP32-WROOM-32E-N4 -> ESP32-WROOM-32E
- U2: value LMV321 -> MCP73831; device My-OpAmps:SOT-23-5 -> My-ICs:SOT-23-5
- U3: value MCP73831 -> LMV321; device My-ICs:SOT-23-5 -> My-OpAmps:SOT-23-5
- U4: value TLV75530PDBVR -> DS3231-SO16; device My-LDOs:SOT-23-5 -> My-ICs:SOIC-16W_(SO16)
- U5: value DS3231-SO16 -> 1117-3.3V; device My-ICs:SOIC-16W_(SO16) -> My-LDOs:SOT-223-3
- moved C18 100.1 mm to (1.33, 38.6), turned to 270 degrees
- moved R6 91.2 mm to (11.6, 13.8), turned to 90 degrees
- moved Q1 86.8 mm to (13.2, 18.3)
- moved R7 86.1 mm to (16.8, 13.8), turned to 90 degrees
- moved R13 78.6 mm to (48.3, 40.3), turned to 270 degrees
- moved R15 76.3 mm to (32.0, 13.4), turned to 90 degrees
- moved C11 73.4 mm to (22.5, 35.0), flipped to the top, turned to 180 degrees
- moved R18 72.5 mm to (36.2, 30.2), turned to 180 degrees
- moved U2 71.6 mm to (25.2, 18.4), turned to 180 degrees
- moved R19 69.0 mm to (36.2, 31.8)
- moved C6 68.4 mm to (35.5, 40.4), turned to 90 degrees
- moved C14 68.0 mm to (25.8, 27.7), flipped to the top, turned to 270 degrees
- moved D1 58.0 mm to (43.6, 35.6)
- moved R16 56.5 mm to (36.2, 33.3)
- moved C15 55.4 mm to (4.69, 32.8), turned to 180 degrees
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Connections:
- net ESP32_UART_RX_USB renamed USB_TX
- net ESP32_UART_TX_USB renamed USB_RX
- removed net !DISPLAY_OLED_RESET: DS1.14, DS1.15, R24.1
- removed net ESP32_ADC_BATTERY_SUPPLY_MONITOR: R18.1, R19.2, SOC1.4
- removed net ESP32_GPIO_PROG_ENABLE: C7.1, C8.1, CN4.10, Q2.3, R10.2, SOC1.3
- removed net ESP32_GPIO_PROG_MODE: C11.1, Q3.3, R12.2, SOC1.25
- removed net ESP32_I2C_SCL: DS1.18, R22.1, SOC1.36, U5.16
- removed net ESP32_I2C_SDA: DS1.19, DS1.20, R21.1, SOC1.33, U5.15
- removed net ESP32_USB_RTS: Q2.2, R11.1, U1.24
- removed net JTAG_TCK: CN4.4, SOC1.16
- removed net JTAG_TDI: CN4.8, SOC1.14
- removed net JTAG_TDO: CN4.6, SOC1.23
- removed net JTAG_TMS: CN4.2, SOC1.13
- removed net N$10: C2.1, CN1.G1, CN1.G2, CN1.G3, CN1.G4, R4.2
- removed net N$13: Q2.1, R8.1
- removed net N$16: Q3.1, R11.2
- removed net N$18: R5.2, U1.9
- removed net N$19: R1.2, U1.5
- removed net N$20: Q3.2, R8.2, U1.28
- removed net N$21: CN1.B5, R9.1
- removed net N$22: R2.2, U1.4
- removed net USB_N: CN1.A7, CN1.B7, R1.1
- removed net USB_P: CN1.A6, CN1.B6, R2.1
- new net ESP32_ADC_BATTERY_SMONITOR: R18.1, R19.2, SOC1.7
- new net ESP32_PROG_ENABLE: C3.1, C5.1, Q1.3, R5.2, SOC1.3
- new net ESP32_PROG_MODE: C8.1, Q2.3, R7.2, SOC1.25
- new net I2C_SCL: CN2.3, R9.1, SOC1.36, U4.16
- new net I2C_SDA: CN2.4, R8.1, SOC1.33, U4.15
- new net N$2: CN1.A5, R4.1
- new net N$79: C1.2, CN1.SHLD1, CN1.SHLD2, CN1.SHLD3, CN1.SHLD4, R1.1
- new net USB_DTR: Q2.2, R2.2, U1.28
- new net USB_RTS: Q1.2, R6.2, U1.24
- net 0V: now also C1.1, C10.1, C12.1, C13.1, C15.2, C2.1, C3.2, C5.2, C7.1, CN1.GND, CN1.GND2, CN2.1, CN4.2, Q3.2, R1.2, R10.1, R11.2, R17.2, R4.2, U4.10, U4.11, U4.12, U4.13, U4.5, U4.6, U4.7, U4.8, U4.9, U5.1; no longer C1.2, C10.2, C12.2, C13.2, C15.1, C2.2, C21.2, C3.1, C5.1, C7.2, CN1.A1, CN1.A12, CN1.B1, CN1.B12, CN4.3, CN4.5, CN4.9, CN6.-, DS1.1, DS1.10, DS1.12, DS1.29, DS1.30, DS1.8, Q1.2, R16.2, R17.1, R23.1, R25.1, R4.1, R6.2, R9.2, U4.2, U5.10, U5.11, U5.12, U5.13, U5.5, U5.6, U5.7, U5.8, U5.9
- net 3.3V: now also C10.2, C11.1, C12.2, C13.2, C19.1, C6.1, C7.2, CN2.2, R7.1, R8.2, R9.2, U3.5, U4.2, U5.4; no longer C1.1, C10.1, C13.1, C14.1, C15.2, C21.1, C5.2, CN4.1, DS1.11, DS1.6, DS1.9, R10.1, R12.1, R21.2, R22.2, R24.2, U2.5, U4.5
- net ESP32_ADC_TASK_FEEDBACK_MONITOR: now also C15.1, R12.2, SOC1.12; no longer C6.1, R13.2, SOC1.11
- net ESP32_GPIO_BATTERY_CHARGING_STATUS: now also SOC1.11, U2.1; no longer SOC1.6, U3.1
- net ESP32_GPIO_EXTERNAL_SUPPLY_MONITOR: now also R16.2, R17.1, SOC1.6; no longer R15.2, R16.1, SOC1.5, U1.8
- net ESP32_GPIO_TASK_CONTROLLER: now also R11.1, R13.2, SOC1.10; no longer R6.1, R7.2, SOC1.8
- net N$1: now also CN1.B5, R3.1; no longer C19.1, DS1.27
- net N$11: now also R15.2; no longer R20.2
- net N$12: now also R12.1, U3.1, U3.4; no longer R13.1, U2.1, U2.4
- net N$14: now also CN6.2; no longer CN2.2
- net N$15: now also CN6.3; no longer CN2.3
- net N$26: now also R10.2, U2.5; no longer R14.2, U3.5
- net N$3: now also CN1.A7, CN1.B7, U1.5; no longer DS1.13, DS1.16, DS1.17, DS1.21, DS1.22, DS1.23, DS1.24, DS1.25, R25.2
- net N$4: now also U3.3; no longer U2.3
- net N$41: now also Q3.1, R13.1; no longer Q1.1, R7.1
- net N$42: now also Q3.3; no longer Q1.3
- net N$5: now also CN6.1; no longer CN2.1
- net N$6: now also CN1.A6, CN1.B6, U1.4; no longer DS1.26, R23.2
- net N$7: now also Q1.1, R2.1; no longer C17.1, DS1.28
- net N$8: now also Q2.1, R6.1; no longer CN1.A5, R3.1
- net P$1: now also U2.3; no longer U3.3
- net RTC_VBAT: now also C14.1, CN4.1, U4.14; no longer C18.1, CN6.+, U5.14
- net VBUS: now also C2.2, CN1.VBUS1, CN1.VBUS2, R14.2, R16.1, U1.8, U2.4; no longer C3.2, CN1.A4, CN1.A9, CN1.B4, CN1.B9, R17.2, R20.1, U3.4
- net VSYS: now also C17.1, C18.1, U5.3; no longer C12.1, U4.1, U4.3
Routing:
- net 3.3V: track 6.87 -> 172.5 mm, vias 0 -> 8
- net 0V: track 10.1 -> 102.5 mm, vias 0 -> 32
- net VSYS: track 0.00 -> 91.7 mm, vias 0 -> 1
- net VBUS: track 20.0 -> 87.7 mm, vias 0 -> 2
- net P$1: track 0.00 -> 67.0 mm, vias 0 -> 1
- net ESP32_ADC_TASK_FEEDBACK_MONITOR: track 0.00 -> 52.1 mm, vias 0 -> 2
- net ESP32_PROG_ENABLE: track 0.00 -> 50.6 mm, vias 0 -> 2
- net USB_RX: track 0.00 -> 37.3 mm, vias 0 -> 1
- net USB_TX: track 0.00 -> 35.7 mm, vias 0 -> 1
- net I2C_SDA: track 0.00 -> 31.3 mm
- net RTC_VBAT: track 0.00 -> 29.7 mm
- net N$79: track 0.00 -> 26.1 mm
- net USB_RTS: track 0.00 -> 26.1 mm, vias 0 -> 1
- net ESP32_GPIO_TASK_CONTROLLER: track 0.00 -> 26.0 mm, vias 0 -> 2
- net JTAG_TMS: track 25.5 -> 0.00 mm
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- added copper zone on layer 1, net 0V
- added copper zone on layer 16, net 0V
Other:
- outline, holes or cut-outs redrawn
- board text added: "GND"
- board text added: "INPUT MONITOR"
- board text added: "It's Time, Do!"
- board text added: "PCB v1.0"
- board text removed: "INPUT"
