File: Hardware/0. Project/It-s Time, Do.sch (EAGLE design)
At the start: 67 parts, among them CN1 CELL-CONNECTOR, CN13 USB 3.2 Gen 2 Type C Receptac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, CN2 2P-MINI-FIT-JR, CN3 3P-MINI-FIT-JR, CN4 JTAG, CN5 CR-1220, Q1 P-FET-ENHANCEMENT-SI2369BDS, Q14 NPN-BC817, Q15 NPN-BC817, Q3 BC817, U1 MCP73831, U12 CP2102N, U2 TLV75530PDBVR, U3 LMV321, U8 DS3231-SO16

Commit message: Schematic WIP
Parts:
- removed C75, C76: 1nF, My-RLC:C_0603
- removed R78: DNP, My-RLC:R_0603
- added C11, C12: 1nF, My-RLC:C_0603
- R76, R77: value 22R -> 22R (5%)
- R82: value 22k -> 10k (5%)
- R83, R85: value 4k7 -> 4k7 (5%)
Connections:
- net ADC_BATTERY_VOLTAGE renamed ESP32_ADC_BATTERY_SUPPLY_MONITOR
- net GPIO_BATTERY_CHARGING_STATUS renamed ESP32_GPIO_BATTERY_CHARGING_STATUS
- removed net ESP32_GPIO_USB_DETECT: R71.2, R72.1
- removed net ESP32_GPIO_USB_DETECT1: U12.VBUS
- removed net ESP32_PROG_ENABLE: C44.1, C75.1, CN4.!RST, Q14.C, R86.2, SOC1.EN
- removed net ESP32_PROG_MODE: C76.1, Q15.C, R87.2, SOC1.IO0
- removed net ESP32_SERIAL1_UART_RX: SOC1.IO16(RXD2)
- removed net ESP32_SERIAL1_UART_TX: SOC1.IO17(TXD2)
- removed net ESP32_SERIAL2_UART_RX: SOC1.IO35
- removed net ESP32_SERIAL2_UART_TX: SOC1.IO33
- removed net ESP32_SERIAL_UART_RX: SOC1.IO3(RXD0)
- removed net ESP32_SERIAL_UART_TX: SOC1.IO1(TXD0)
- removed net N$48: R82.1, U12.!RST
- removed net N$49: R78.2, U12.!SUSPEND
- new net ESP32_GPIO_EXTERNAL_SUPPLY_MONITOR: R71.2, R72.1, U12.VBUS
- new net ESP32_GPIO_PROG_ENABLE: C11.1, C44.1, CN4.!RST, Q14.C, R86.2, SOC1.EN
- new net ESP32_GPIO_PROG_MODE: C12.1, Q15.C, R87.2, SOC1.IO0
- new net N$17: C72.2, U12.GND
- new net N$18: R82.2, U12.!RST
- net 0V: now also C11.2, C12.2; no longer C72.2, C75.2, C76.2, R78.1, U12.GND
- net 3.3V: now also R82.1; no longer R82.2
- net ESP32_UART_RX_USB: now also SOC1.IO3(RXD0)
- net ESP32_UART_TX_USB: now also SOC1.IO1(TXD0)
- net ESP32_USB_RTS: now also R85.1; no longer R85.2
- net N$16: now also R85.2; no longer R85.1
Other:
- note added: "!JTAG/RST"
- note removed: "( !JTAG/RST )"
- moved on the sheet: C1, C10, C17, C2, C3, C4, C44, C45, C46, C5, C6, C67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

Commit message: Schematic WIP
Parts:
- removed C44, C45: 10uF, My-RLC:C_0603
- removed C46, C72: 100nF, My-RLC:C_0603
- removed Q14, Q15: NPN-BC817, My-Transistors:NPN-BC817
- removed R71: 24k, My-RLC:R_0603
- removed R76, R77: 22R (5%), My-RLC:R_0603
- removed R82: 10k (5%), My-RLC:R_0603
- removed R83, R85: 4k7 (5%), My-RLC:R_0603
- removed R86, R87: 10k (1%), My-RLC:R_0603
- removed U12: CP2102N, My-ICs:CP2102N
- removed U8: DS3231-SO16, My-ICs:DS3231-SO16
- added C13, C15: 10uF, My-RLC:C_0603
- added C14: 1nF, My-RLC:C_0603
- added C16: 10nF, My-RLC:C_0603
- added C21: 100nF, My-RLC:C_0603
- added Q2: NPN-BC817, My-Transistors:NPN-BC817
- added Q4: BC817, My-Transistors:NPN-BC817
- added R14: 47R, My-RLC:R_0603
- added R17, R19, R20: 4k7 (5%), My-RLC:R_0603
- added R21, R22: 10k (5%), My-RLC:R_0603
- added R25, R26: 22R (5%), My-RLC:R_0603
- added U4: LMV321, My-OpAmps:SINGLE
- added U5: CP2102N, My-ICs:CP2102N
- C1: PARTNO GRM155R71H104KE14D -> *; PN C0603C104M5RACTU -> (none)
- C10: value 100nF -> 100uF x 10V; device My-RLC:C_0603 -> My-RLC:CP_5MM; PARTNO * -> (none)
- C12: value 1nF -> 100nF; PARTNO GRJ155R60J106ME11D -> GRM155R71H104KE14D; PN GRM188R61A106ME69D -> C0603C104M5RACTU
- C2: value 10nF -> 1uF; PARTNO (none) -> *
- C3: value 100nF -> 10uF; PARTNO * -> GRM155R71H104KE14D; PN (none) -> C0603C104M5RACTU; SPICEPREFIX (none) -> C
- C4: PARTNO GRM155R71H104KE14D -> GRJ155R60J106ME11D; PN C0603C104M5RACTU -> GRM188R61A106ME69D
- C5: SPICEPREFIX C -> (none)
- C6: value 10uF -> 100nF; PARTNO GRM155R71H104KE14D -> *; PN C0603C104M5RACTU -> (none)
- C7: value 100uF x 10V -> 100nF; device My-RLC:CP_5MM -> My-RLC:C_0603; PARTNO (none) -> *
- C8: value 1uF -> 10uF; PARTNO * -> GRM155R71H104KE14D; PN (none) -> C0603C104M5RACTU
- C9: PARTNO * -> GRM155R71H104KE14D; PN (none) -> C0603C104M5RACTU
- CN1: value CELL-CONNECTOR -> CR-1220; device My-Battery:CELL-CONNECTOR -> My-Battery:CR-1220; PARTNO (none) -> *
- CN2: value 2P-MINI-FIT-JR -> CELL-CONNECTOR; device My-Connectors:2P-MINI-FIT-JR -> My-Battery:CELL-CONNECTOR
- CN3: value 3P-MINI-FIT-JR -> JTAG; device My-Connectors:3P-MINI-FIT-JR -> My-Connectors:JTAG; PARTNO (none) -> FTSH-105-01-L-DV-K
- CN4: value JTAG -> 2P-MINI-FIT-JR; device My-Connectors:JTAG -> My-Connectors:2P-MINI-FIT-JR; PARTNO FTSH-105-01-L-DV-K -> (none)
- CN5: value CR-1220 -> 3P-MINI-FIT-JR; device My-Battery:CR-1220 -> My-Connectors:3P-MINI-FIT-JR; PARTNO * -> (none)
- Q3: value BC817 -> NPN-BC817; PARTNO (none) -> PMMT491A,215; PN BC817K-16HR -> (none)
- R1: value 47R -> 10k (5%)
- R11: value 4k7 (5%) -> 24k; PARTNO (none) -> RC0402FR-0724KL; PN RC0603JR-074K7L -> RC0603JR-0724KL
- R13: value 10k (5%) -> 22K (5%); PARTNO (none) -> *; PN RC0603JR-0710KL -> (none)
- R15, R16: value 1M -> 10k (1%); PARTNO * -> RC0402FR-0710KL; PN (none) -> RC0603JR-0710KL
- R2, R3: value 4k7 (5%) -> 10k (5%)
- R5, R6: value 10k (5%) -> 4k7 (5%)
- R7: value 10k (5%) -> 100R (5%)
- R8: value 4k7 -> 1M
- R9: value 100R (5%) -> 1M; PARTNO (none) -> *
- U1: value MCP73831 -> DS3231-SO16; device My-ICs:MCP73831T-2ACI/OT -> My-ICs:DS3231-SO16; PARTNO * -> (none)
- U3: value LMV321 -> MCP73831; device My-OpAmps:SINGLE -> My-ICs:MCP73831T-2ACI/OT; PARTNO (none) -> *
- renumbered C67 to C20, C69 to C19, C71 to C18, CN13 to CN6, D7 to D2, R62 to R24, R63 to R23, R65 to R18, R72 to R12
Connections:
- removed net ESP32_USB_DTR: Q15.E, R83.2, U12.DTR
- removed net N$17: C72.2, U12.GND
- removed net N$9: CN5.+, U8.VBAT
- new net N$20: Q2.E, R19.2, U5.DTR
- new net RTC_VBAT: C4.1, CN1.+, U1.VBAT
- net !DISPLAY_OLED_RESET: now also R2.1; no longer R5.1
- net 0V: now also C10.-, C13.2, C14.2, C15.2, C16.2, C17.2, C21.2, C7.1, CN2.-, CN3.GND, CN3.GND2, CN3.GND3, CN4-2.P$1, Q4.E, R13.1, R21.2, R3.1, R9.1, U1.GND, U3.VSS, U4G$1.V-, U5.GND; no longer C10.2, C17.1, C44.2, C45.2, C46.2, C7.-, CN2-2.P$1, CN4.GND, CN4.GND2, CN4.GND3, CN5.-, Q3.E, R13.2, R16.1, R7.1, R8.1, U1.VSS, U3G$1.V-, U8.GND
- net 3.3V: now also C12.1, C13.1, C17.1, C2.1, C21.1, C7.2, CN3.VDD, R1.2, R15.1, R16.1, R22.1, U1.VDD, U4G$1.V+, U5.REGIN, U5.VDD; no longer C10.1, C17.2, C4.1, C45.1, C46.1, C72.1, CN4.VDD, R3.2, R82.1, R86.1, R87.1, U12.REGIN, U12.VDD, U3G$1.V+, U8.VDD
- net ESP32_ADC_BATTERY_SUPPLY_MONITOR: now also R8.1, R9.2, SOC1.IO36; no longer R15.1, R16.2
- net ESP32_ADC_TASK_FEEDBACK_MONITOR: now also C16.1, R14.2; no longer C2.1, R1.2
- net ESP32_GPIO_BATTERY_CHARGING_STATUS: now also SOC1.IO34, U3.STAT; no longer U1.STAT
- net ESP32_GPIO_EXTERNAL_SUPPLY_MONITOR: now also R11.2, SOC1.IO39, U5.VBUS; no longer R71.2, U12.VBUS
- net ESP32_GPIO_PROG_ENABLE: now also C14.1, C15.1, CN3.!RST, Q3.C, R16.2; no longer C11.1, C44.1, CN4.!RST, Q14.C, R86.2
- net ESP32_GPIO_PROG_MODE: now also C11.1, Q2.C, R15.2; no longer C12.1, Q15.C, R87.2
- net ESP32_GPIO_TASK_CONTROLLER: now also R20.2, R21.1; no longer R11.2, R13.1
- net ESP32_I2C_SCL: now also R5.1, U1.SCL; no longer R3.1, U8.SCL
- net ESP32_I2C_SDA: now also R6.1, U1.SDA; no longer R2.1, U8.SDA
- net ESP32_UART_RX_USB: now also U5.TXD; no longer U12.TXD
- net ESP32_UART_TX_USB: now also U5.RXD; no longer U12.RXD
- net ESP32_USB_RTS: now also Q3.E, R17.1, U5.RTS; no longer Q14.E, R85.1, U12.RTS
- net JTAG_TCK: now also CN3.TCK; no longer CN4.TCK
- net JTAG_TDI: now also CN3.TDI; no longer CN4.TDI
- net JTAG_TDO: now also CN3.TDO; no longer CN4.TDO
- net JTAG_TMS: now also CN3.TMS; no longer CN4.TMS
- net N$1: now also C3.1; no longer C5.1
- net N$11: now also R7.2; no longer R9.2
- net N$12: now also R14.1, U4-A.-IN, U4-A.OUT; no longer R1.1, U3-A.-IN, U3-A.OUT
- net N$13: now also Q3.B, R19.1; no longer Q14.B, R83.1
- net N$14: now also CN5-2.P$1; no longer CN3-2.P$1
- net N$15: now also CN5-3.P$1; no longer CN3-3.P$1
- net N$16: now also Q2.B, R17.2; no longer Q15.B, R85.2
- net N$18: now also R22.2, U5.!RST; no longer R82.2, U12.!RST
- net N$19: now also R25.2, U5.D-; no longer R76.2, U12.D-
- net N$2: now also R1.1; no longer R6.1
- net N$22: now also R26.2, U5.D+; no longer R77.2, U12.D+
- net N$26: now also R13.2, U3.PROG; no longer R8.2, U1.PROG
- net N$3: now also R3.2; no longer R7.2
- net N$4: now also CN4-1.P$1, U4-A.+IN; no longer CN2-1.P$1, U3-A.+IN
- net N$41: now also Q4.B, R20.1; no longer Q3.B, R11.1
- net N$42: now also Q4.C; no longer Q3.C
- net N$5: now also CN5-1.P$1; no longer CN3-1.P$1
- net N$7: now also C5.1; no longer C6.1
- net P$1: now also CN2.+, R8.2, U3.VBAT; no longer CN1.+, R15.2, U1.VBAT
- net USB_N: now also CN6.DN1, CN6.DN2, R25.1; no longer R76.1
- net USB_P: now also CN6.DP1, CN6.DP2, R26.1; no longer R77.1
- net VBUS: now also R11.1, R7.1, U3.VDD; no longer R71.1, R9.1, U1.VDD
- net VSYS: now also C10.+, C6.1; no longer C3.1, C7.+
Other:
- note added: "I-REG = 45mA"
- note removed: "I-REG = 213mA"
- moved on the sheet: C1, C11, C12, C17, C2, C3, C4, C5, C6, C8, C9, CN1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

Commit message: Schematic WIP
Parts:
- C1: PARTNO * -> GRM155R71H104KE14D; PN (none) -> C0603C104M5RACTU
- C10: value 100uF x 10V -> 100nF; device My-RLC:CP_5MM -> My-RLC:C_0603; PARTNO (none) -> GRM155R71H104KE14D; PN (none) -> C0603C104M5RACTU
- C12: value 100nF -> 100uF x 10V; device My-RLC:C_0603 -> My-RLC:CP_5MM; PARTNO GRM155R71H104KE14D -> (none); PN C0603C104M5RACTU -> (none)
- C13: value 10uF -> 100nF; PARTNO GRJ155R60J106ME11D -> GRM155R71H104KE14D; PN GRM188R61A106ME69D -> C0603C104M5RACTU
- C14: value 1nF -> 10uF; PARTNO GRJ155R60J106ME11D -> GRM155R71H104KE14D; PN GRM188R61A106ME69D -> C0603C104M5RACTU
- C15: value 10uF -> 100nF; PARTNO GRJ155R60J106ME11D -> *; PN GRM188R61A106ME69D -> (none)
- C16: value 10nF -> 100nF; PARTNO (none) -> *
- C17: value 100nF -> 10uF; PARTNO * -> GRM155R71H104KE14D; PN (none) -> C0603C104M5RACTU
- C18: PN (none) -> GRM188R61A106ME69D
- C19: value 100nF -> 10uF; PN (none) -> C0603C104M5RACTU; SPICEPREFIX (none) -> C
- C2: value 1uF -> 4.7nF; PARTNO * -> GRM155R72A472KA01D
- C20: value 4.7nF -> 1uF; PARTNO GRM155R72A472KA01D -> *
- C21: PARTNO GRM155R71H104KE14D -> *; PN C0603C104M5RACTU -> (none)
- C3: value 10uF -> 100nF; PN C0603C104M5RACTU -> (none); SPICEPREFIX C -> (none)
- C4: PN GRM188R61A106ME69D -> (none)
- C5: value 10uF -> 100nF; PARTNO GRM155R71H104KE14D -> *; PN C0603C104M5RACTU -> (none)
- C6: value 100nF -> 10nF; PARTNO * -> (none)
- C7: value 100nF -> 10uF; PARTNO * -> GRJ155R60J106ME11D; PN (none) -> GRM188R61A106ME69D
- C8: value 10uF -> 1nF; PARTNO GRM155R71H104KE14D -> GRJ155R60J106ME11D; PN C0603C104M5RACTU -> GRM188R61A106ME69D
- C9: value 100nF -> 10uF; PARTNO GRM155R71H104KE14D -> GRJ155R60J106ME11D; PN C0603C104M5RACTU -> GRM188R61A106ME69D
- CN1: value CR-1220 -> USB 3.2 Gen 2 Type C Receptacle; device My-Battery:CR-1220 -> My-Connectors:USB-C; PARTNO * -> USB4080-03-A
- CN2: value CELL-CONNECTOR -> 3P-MINI-FIT-JR; device My-Battery:CELL-CONNECTOR -> My-Connectors:3P-MINI-FIT-JR
- CN3: value JTAG -> 2P-MINI-FIT-JR; device My-Connectors:JTAG -> My-Connectors:2P-MINI-FIT-JR; PARTNO FTSH-105-01-L-DV-K -> (none)
- CN4: value 2P-MINI-FIT-JR -> JTAG; device My-Connectors:2P-MINI-FIT-JR -> My-Connectors:JTAG; PARTNO (none) -> FTSH-105-01-L-DV-K
- CN5: value 3P-MINI-FIT-JR -> CELL-CONNECTOR; device My-Connectors:3P-MINI-FIT-JR -> My-Battery:CELL-CONNECTOR
- CN6: value USB 3.2 Gen 2 Type C Receptacle -> CR-1220; device My-Connectors:USB-C -> My-Battery:CR-1220; PARTNO USB4080-03-A -> *
- D1: value SCHOTTKY-SS16 -> FM4004; PN (none) -> FM4004W-W
- D2: value FM4004 -> SCHOTTKY-SS16; PN FM4004W-W -> (none)
- Q1: value P-FET-ENHANCEMENT-SI2369BDS -> BC817; device My-Transistors:P-FET-ENHANCEMENT-SI2369BDS -> My-Transistors:NPN-BC817; PN (none) -> BC817K-16HR
- Q4: value BC817 -> P-FET-ENHANCEMENT-SI2369BDS; device My-Transistors:NPN-BC817 -> My-Transistors:P-FET-ENHANCEMENT-SI2369BDS; PN BC817K-16HR -> (none)
- R1, R2: value 10k (5%) -> 22R (5%); PARTNO (none) -> RC0402FR-1322RL; PN (none) -> RC0603JR-0724KL
- R10: value 10k (5%) -> 10k (1%); PARTNO (none) -> RC0402FR-0710KL; PN (none) -> RC0603JR-0710KL
- R11: value 24k -> 4k7 (5%); PARTNO RC0402FR-0724KL -> RC0402JR-074K7L; PN RC0603JR-0724KL -> RC0603JR-074K7L
- R12: value 47k -> 10k (1%); PARTNO RC0402FR-0747KL -> RC0402FR-0710KL; PN RC0603JR-1047KL -> RC0603JR-0710KL
- R13: value 22K (5%) -> 47R; PARTNO * -> (none)
- R14: value 47R -> 22K (5%); PARTNO (none) -> *
- R15: value 10k (1%) -> 24k; PARTNO RC0402FR-0710KL -> RC0402FR-0724KL; PN RC0603JR-0710KL -> RC0603JR-0724KL
- R16: value 10k (1%) -> 47k; PARTNO RC0402FR-0710KL -> RC0402FR-0747KL; PN RC0603JR-0710KL -> RC0603JR-1047KL
- R17: value 4k7 (5%) -> 10k (5%); PARTNO RC0402JR-074K7L -> (none); PN RC0603JR-074K7L -> (none)
- R18: value 5k1 -> 1M; PARTNO AC0402FR-075K1L -> *
- R19: value 4k7 (5%) -> 1M; PARTNO RC0402JR-074K7L -> *; PN RC0603JR-074K7L -> (none)
- R20: value 4k7 (5%) -> 100R (5%); PN RC0603JR-074K7L -> (none)
- R21: value 10k (5%) -> 4k7 (5%); PN RC0603JR-0710KL -> (none)
- R22: value 10k (5%) -> 4k7 (5%); PARTNO RC0402FR-0722KL -> (none); PN RC0603JR-0722KL -> (none)
- R23: value 1M -> 390k (1%); PARTNO RC0402JR-071ML -> (none)
- R24: value 5k1 -> 10k (5%); PARTNO AC0402FR-075K1L -> (none)
- R25, R26: value 22R (5%) -> 10k (5%); PARTNO RC0402FR-1322RL -> (none); PN RC0603JR-0724KL -> (none)
- R3: value 10k (5%) -> 5k1; PARTNO (none) -> AC0402FR-075K1L
- R4: value 390k (1%) -> 1M; PARTNO (none) -> RC0402JR-071ML
- R5: value 4k7 (5%) -> 10k (5%); PARTNO (none) -> RC0402FR-0722KL; PN (none) -> RC0603JR-0722KL
- R6: value 4k7 (5%) -> 10k (5%); PN (none) -> RC0603JR-0710KL
- R7: value 100R (5%) -> 4k7 (5%); PN (none) -> RC0603JR-074K7L
- R8: value 1M -> 4k7 (5%); PARTNO * -> RC0402JR-074K7L; PN (none) -> RC0603JR-074K7L
- R9: value 1M -> 5k1; PARTNO * -> AC0402FR-075K1L
- U1: value DS3231-SO16 -> CP2102N; device My-ICs:DS3231-SO16 -> My-ICs:CP2102N; PARTNO (none) -> CP2102N-A02-GQFN28; PN (none) -> CP2102N-A02-GQFN28
- U2: value TLV75530PDBVR -> LMV321; device My-LDOs:TLV75530PDBVR -> My-OpAmps:SINGLE; PARTNO * -> (none)
- U4: value LMV321 -> TLV75530PDBVR; device My-OpAmps:SINGLE -> My-LDOs:TLV75530PDBVR; PARTNO (none) -> *
- U5: value CP2102N -> DS3231-SO16; device My-ICs:CP2102N -> My-ICs:DS3231-SO16; PARTNO CP2102N-A02-GQFN28 -> (none); PN CP2102N-A02-GQFN28 -> (none)
Connections:
- net !DISPLAY_OLED_RESET: now also R24.1; no longer R2.1
- net 0V: now also C10.2, C12.-, C15.1, C18.2, C19.2, C2.1, C20.2, C3.1, C4.1, C7.2, CN1.GND_A, CN1.GND_B, CN3-2.P$1, CN4.GND, CN4.GND2, CN4.GND3, CN5.-, CN6.-, Q1.E, R14.1, R16.2, R17.1, R19.1, R23.1, R25.1, R3.2, R4.2, R6.2, R9.2, U2G$1.V-, U4.GND; no longer C10.-, C12.2, C15.2, C18.1, C19.1, C2.2, C20.1, C3.2, C4.2, C7.1, CN1.-, CN2.-, CN3.GND, CN3.GND2, CN3.GND3, CN4-2.P$1, CN6.GND_A, CN6.GND_B, Q4.E, R10.1, R12.2, R13.1, R18.2, R21.2, R23.2, R24.2, R3.1, R4.1, R9.1, U2.GND, U4G$1.V-
- net 3.3V: now also C10.1, C14.1, C15.2, C20.1, C5.1, CN4.VDD, R10.1, R12.1, R21.2, R22.2, R24.2, R26.2, R5.1, U1.REGIN, U2G$1.V+, U4.OUT; no longer C12.1, C17.1, C2.1, C7.2, C8.1, CN3.VDD, R1.2, R15.1, R16.1, R2.2, R22.1, R5.2, R6.2, U2.OUT, U4G$1.V+, U5.REGIN
- net ESP32_ADC_BATTERY_SUPPLY_MONITOR: now also R18.1, R19.2; no longer R8.1, R9.2
- net ESP32_ADC_TASK_FEEDBACK_MONITOR: now also C6.1, R13.2, SOC1.IO26; no longer C16.1, R14.2
- net ESP32_GPIO_EXTERNAL_SUPPLY_MONITOR: now also R15.2, R16.1, U1.VBUS; no longer R11.2, R12.1, U5.VBUS
- net ESP32_GPIO_PROG_ENABLE: now also C7.1, C8.1, CN4.!RST, Q2.C, R10.2; no longer C14.1, C15.1, CN3.!RST, Q3.C, R16.2
- net ESP32_GPIO_PROG_MODE: now also Q3.C, R12.2; no longer Q2.C, R15.2
- net ESP32_GPIO_TASK_CONTROLLER: now also R6.1, R7.2, SOC1.IO32; no longer R20.2, R21.1
- net ESP32_I2C_SCL: now also R22.1, U5.SCL; no longer R5.1, U1.SCL
- net ESP32_I2C_SDA: now also R21.1, U5.SDA; no longer R6.1, U1.SDA
- net ESP32_UART_RX_USB: now also U1.TXD; no longer U5.TXD
- net ESP32_UART_TX_USB: now also U1.RXD; no longer U5.RXD
- net ESP32_USB_RTS: now also Q2.E, R11.1, U1.RTS; no longer Q3.E, R17.1, U5.RTS
- net JTAG_TCK: now also CN4.TCK; no longer CN3.TCK
- net JTAG_TDI: now also CN4.TDI; no longer CN3.TDI
- net JTAG_TDO: now also CN4.TDO; no longer CN3.TDO
- net JTAG_TMS: now also CN4.TMS; no longer CN3.TMS
- net N$1: now also C19.1; no longer C3.1
- net N$10: now also C2.2, CN1.SHIELD, R4.1; no longer C20.2, CN6.SHIELD, R23.1
- net N$11: now also Q4.G, R20.2; no longer Q1.G, R7.2
- net N$12: now also R13.1, U2-A.-IN, U2-A.OUT; no longer R14.1, U4-A.-IN, U4-A.OUT
- net N$13: now also Q2.B, R8.1; no longer Q3.B, R19.1
- net N$14: now also CN2-2.P$1; no longer CN5-2.P$1
- net N$15: now also CN2-3.P$1; no longer CN5-3.P$1
- net N$16: now also Q3.B, R11.2; no longer Q2.B, R17.2
- net N$18: now also R5.2, U1.!RST; no longer R22.2, U5.!RST
- net N$19: now also R1.2, U1.D-; no longer R25.2, U5.D-
- net N$2: now also R26.1; no longer R1.1
- net N$20: now also Q3.E, R8.2, U1.DTR; no longer Q2.E, R19.2, U5.DTR
- net N$21: now also CN1.CC2, R9.1; no longer CN6.CC2, R18.1
- net N$22: now also R2.2, U1.D+; no longer R26.2, U5.D+
- net N$26: now also R14.2; no longer R13.2
- net N$3: now also R25.2; no longer R3.2
- net N$4: now also CN3-1.P$1, U2-A.+IN; no longer CN4-1.P$1, U4-A.+IN
- net N$41: now also Q1.B, R7.1; no longer Q4.B, R20.1
- net N$42: now also D1.A, Q1.C; no longer D2.A, Q4.C
- net N$5: now also CN2-1.P$1; no longer CN5-1.P$1
- net N$6: now also R23.2; no longer R4.2
- net N$7: now also C17.1; no longer C5.1
- net N$8: now also CN1.CC1, R3.1; no longer CN6.CC1, R24.1
- net P$1: now also CN5.+, Q4.D, R18.2; no longer CN2.+, Q1.D, R8.2
- net RTC_VBAT: now also C18.1, CN6.+, U5.VBAT; no longer C4.1, CN1.+, U1.VBAT
- net USB_N: now also CN1.DN1, CN1.DN2, R1.1; no longer CN6.DN1, CN6.DN2, R25.1
- net USB_P: now also CN1.DP1, CN1.DP2, R2.1; no longer CN6.DP1, CN6.DP2, R26.1
- net VBUS: now also C3.2, C4.2, CN1.VBUS_A, CN1.VBUS_B, D1.K, D2.A, R15.1, R17.2, R20.1; no longer C18.2, C19.2, CN6.VBUS_A, CN6.VBUS_B, D1.A, D2.K, R10.2, R11.1, R7.1
- net VSYS: now also C12.+, C16.1, D2.K, Q4.S, U4.EN, U4.IN; no longer C10.+, C6.1, D1.K, Q1.S, U2.EN, U2.IN
Other:
- moved on the sheet: C1, C13, C14, C15, C16, C17, C18, C19, C2, C20, C21, C3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

Commit message: Schematic v1.0 release
Parts:
- R13: value 47R -> 47R (5%)
- R15: value 24k -> 24k (5%)
- R16: value 47k -> 47k (5%)
- R18, R19, R4: value 1M -> 1M (1%)
- R3, R9: value 5k1 -> 5k1 (1%)
Connections:
- net 0V: now also C5.1; no longer C5.2
- net 3.3V: now also C5.2; no longer C5.1
Other:
- moved on the sheet: C1, C10, C11, C12, C13, C14, C15, C16, C17, C18, C19, C2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
