File: Hardware/0. Project/It-s Time, Do.sch (EAGLE design)
At the start: 67 parts, among them CN1 USB 3.2 Gen 2 Type C Receptac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, CN2 3P-MINI-FIT-JR, CN3 2P-MINI-FIT-JR, CN4 JTAG, CN5 CELL-CONNECTOR, CN6 CR-1220, Q1 BC817, Q2 NPN-BC817, Q3 NPN-BC817, Q4 P-FET-ENHANCEMENT-SI2369BDS, U1 CP2102N, U2 LMV321, U3 MCP73831, U4 TLV75530PDBVR, U5 DS3231-SO16

Commit message: Board design WIP
Connections:
- net 0V: now also C2.2, R4.1; no longer C2.1, R4.2
- net N$10: now also C2.1, R4.2; no longer C2.2, R4.1
Other:
- moved on the sheet: C2, R4
Changed lines of the file:
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@@
 <part name="R21" library="My-RLC" library_urn="urn:adsk.eagle:library:35509816" deviceset="R_" device="0603" package3d_urn="urn:adsk.eagle:package:35509946/1" value="4k7 (5%)"/>
 <part name="R22" library="My-RLC" library_urn="urn:adsk.eagle:library:35509816" deviceset="R_" device="0603" package3d_urn="urn:adsk.eagle:package:35509946/1" value="4k7 (5%)"/>
-<part name="DS1" library="My-Displays" library_urn="urn:adsk.eagle:library:35510881" deviceset="OLED-RAW" device="-0.96&quot;" package3d_urn="urn:adsk.eagle:package:35806502/1" value="0.96&quot; active Area / 128x64 pixels"/>
+<part name="DS1" library="My-Displays" library_urn="urn:adsk.eagle:library:35510881" deviceset="OLED-RAW" device="-0.96&quot;" package3d_urn="urn:adsk.eagle:package:35807155/3" value="0.96&quot; active Area / 128x64 pixels"/>
 <part name="SUPPLY1" library="My-Supply" library_urn="urn:adsk.eagle:library:35531236" deviceset="3.3V" device=""/>
 <part name="C13" library="My-RLC" library_urn="urn:adsk.eagle:library:35509816" deviceset="C_" device="0603" package3d_urn="urn:adsk.eagle:package:35509984/1" value="100nF">
@@
 </instance>
 <instance part="SUPPLY32" gate="G$1" x="38.735" y="182.245" smashed="yes" grouprefs="POWER_SUPPLY"/>
-<instance part="R3" gate="G$1" x="38.735" y="216.535" smashed="yes" rot="R270" grouprefs="POWER_SUPPLY EXTERNAL_USB_POWER_SUPPLY_INPUT">
-<attribute name="PARTNO" x="38.735" y="216.535" size="1.778" layer="96" display="off"/>
-<attribute name="NAME" x="40.8686" y="216.535" size="1.27" layer="95" rot="R270" align="center"/>
-<attribute name="VALUE" x="36.83" y="216.535" size="1.27" layer="96" rot="R270" align="center"/>
-</instance>
-<instance part="R9" gate="G$1" x="101.6" y="216.535" smashed="yes" rot="R270" grouprefs="POWER_SUPPLY EXTERNAL_USB_POWER_SUPPLY_INPUT">
-<attribute name="PARTNO" x="101.6" y="216.535" size="1.778" layer="96" display="off"/>
-<attribute name="NAME" x="103.7336" y="216.535" size="1.27" layer="95" rot="R270" align="center"/>
-<attribute name="VALUE" x="99.695" y="216.535" size="1.27" layer="96" rot="R270" align="center"/>
-</instance>
-<instance part="R4" gate="G$1" x="45.085" y="200.025" smashed="yes" rot="R270" grouprefs="POWER_SUPPLY EXTERNAL_USB_POWER_SUPPLY_INPUT">
-<attribute name="PARTNO" x="45.085" y="200.025" size="1.778" layer="96" display="off"/>
-<attribute name="NAME" x="47.2186" y="200.025" size="1.27" layer="95" rot="R270" align="center"/>
-<attribute name="VALUE" x="43.18" y="200.025" size="1.27" layer="96" rot="R270" align="center"/>
-</instance>
-<instance part="C2" gate="G$1" x="55.245" y="198.755" smashed="yes" rot="R180" grouprefs="POWER_SUPPLY EXTERNAL_USB_POWER_SUPPLY_INPUT">
-<attribute name="PARTNO" x="55.245" y="198.755" size="1.778" layer="96" display="off"/>
-<attribute name="NAME" x="58.3565" y="200.1012" size="1.27" layer="95" rot="R270" align="center"/>
-<attribute name="VALUE" x="52.07" y="200.1266" size="1.27" layer="96" rot="R270" align="center"/>
+<instance part="R3" gate="G$1" x="38.735" y="216.535" smashed="yes" rot="MR270" grouprefs="POWER_SUPPLY EXTERNAL_USB_POWER_SUPPLY_INPUT">
+<attribute name="PARTNO" x="38.735" y="216.535" size="1.778" layer="96" rot="MR0" display="off"/>
+<attribute name="NAME" x="36.6014" y="216.535" size="1.27" layer="95" rot="MR270" align="center"/>
+<attribute name="VALUE" x="40.64" y="216.535" size="1.27" layer="96" rot="MR270" align="center"/>
+</instance>
+<instance part="R9" gate="G$1" x="101.6" y="216.535" smashed="yes" rot="MR270" grouprefs="POWER_SUPPLY EXTERNAL_USB_POWER_SUPPLY_INPUT">
+<attribute name="PARTNO" x="101.6" y="216.535" size="1.778" layer="96" rot="MR0" display="off"/>
+<attribute name="NAME" x="99.4664" y="216.535" size="1.27" layer="95" rot="MR270" align="center"/>
+<attribute name="VALUE" x="103.505" y="216.535" size="1.27" layer="96" rot="MR270" align="center"/>
+</instance>
+<instance part="R4" gate="G$1" x="45.085" y="200.025" smashed="yes" rot="R90" grouprefs="POWER_SUPPLY EXTERNAL_USB_POWER_SUPPLY_INPUT">
+<attribute name="PARTNO" x="45.085" y="200.025" size="1.778" layer="96" rot="R180" display="off"/>
+<attribute name="NAME" x="42.9514" y="200.025" size="1.27" layer="95" rot="R90" align="center"/>
+<attribute name="VALUE" x="46.99" y="200.025" size="1.27" layer="96" rot="R90" align="center"/>
+</instance>
+<instance part="C2" gate="G$1" x="55.245" y="201.295" smashed="yes" grouprefs="POWER_SUPPLY EXTERNAL_USB_POWER_SUPPLY_INPUT">
+<attribute name="PARTNO" x="55.245" y="201.295" size="1.778" layer="96" rot="R180" display="off"/>
+<attribute name="NAME" x="52.1335" y="199.9488" size="1.27" layer="95" rot="R90" align="center"/>
+<attribute name="VALUE" x="58.42" y="199.9234" size="1.27" layer="96" rot="R90" align="center"/>
 </instance>
 <instance part="C4" gate="G$1" x="121.285" y="208.915" smashed="yes" rot="R180" grouprefs="POWER_SUPPLY EXTERNAL_USB_POWER_SUPPLY_INPUT">
@@
 <segment>
 <pinref part="C3" gate="G$1" pin="1"/>
-<pinref part="R4" gate="G$1" pin="2"/>
 <pinref part="R14" gate="G$1" pin="1"/>
 <wire x1="110.49" y1="189.865" x2="110.49" y2="206.375" width="0.1524" layer="91" grouprefs="POWER_SUPPLY EXTERNAL_USB_POWER_SUPPLY_INPUT"/>
-<wire x1="45.085" y1="189.865" x2="45.085" y2="194.945" width="0.1524" layer="91" grouprefs="POWER_SUPPLY EXTERNAL_USB_POWER_SUPPLY_INPUT"/>
 <wire x1="164.465" y1="194.945" x2="164.465" y2="189.865" width="0.1524" layer="91" grouprefs="BATTERY_CHARGE_MANAGEMENT_CONTROLLER POWER_SUPPLY"/>
 <pinref part="U3" gate="G$1" pin="VSS"/>
@@
 <wire x1="164.465" y1="189.865" x2="121.285" y2="189.865" width="0.1524" layer="91" grouprefs="POWER_SUPPLY"/>
 <junction x="38.735" y="189.865" grouprefs="EXTERNAL_USB_POWER_SUPPLY_INPUT POWER_SUPPLY"/>
-<junction x="45.085" y="189.865" grouprefs="EXTERNAL_USB_POWER_SUPPLY_INPUT POWER_SUPPLY"/>
 <wire x1="121.285" y1="189.865" x2="110.49" y2="189.865" width="0.1524" layer="91" grouprefs="EXTERNAL_USB_POWER_SUPPLY_INPUT POWER_SUPPLY"/>
 <wire x1="110.49" y1="189.865" x2="101.6" y2="189.865" width="0.1524" layer="91" grouprefs="EXTERNAL_USB_POWER_SUPPLY_INPUT POWER_SUPPLY"/>
@@
 <wire x1="55.245" y1="189.865" x2="45.085" y2="189.865" width="0.1524" layer="91" grouprefs="EXTERNAL_USB_POWER_SUPPLY_INPUT POWER_SUPPLY"/>
 <wire x1="45.085" y1="189.865" x2="38.735" y2="189.865" width="0.1524" layer="91" grouprefs="EXTERNAL_USB_POWER_SUPPLY_INPUT POWER_SUPPLY"/>
-<pinref part="C2" gate="G$1" pin="1"/>
-<junction x="55.245" y="189.865" grouprefs="EXTERNAL_USB_POWER_SUPPLY_INPUT POWER_SUPPLY"/>
-<wire x1="55.245" y1="189.865" x2="55.245" y2="196.215" width="0.1524" layer="91" grouprefs="POWER_SUPPLY EXTERNAL_USB_POWER_SUPPLY_INPUT"/>
 <wire x1="94.615" y1="211.455" x2="101.6" y2="211.455" width="0.1524" layer="91" grouprefs="POWER_SUPPLY EXTERNAL_USB_POWER_SUPPLY_INPUT"/>
 <wire x1="101.6" y1="211.455" x2="101.6" y2="189.865" width="0.1524" layer="91" grouprefs="POWER_SUPPLY EXTERNAL_USB_POWER_SUPPLY_INPUT"/>
@@
 <junction x="121.285" y="189.865" grouprefs="EXTERNAL_USB_POWER_SUPPLY_INPUT POWER_SUPPLY"/>
 <wire x1="121.285" y1="189.865" x2="121.285" y2="206.375" width="0.1524" layer="91" grouprefs="POWER_SUPPLY EXTERNAL_USB_POWER_SUPPLY_INPUT"/>
+<pinref part="R4" gate="G$1" pin="1"/>
+<wire x1="45.085" y1="194.945" x2="45.085" y2="189.865" width="0.1524" layer="91"/>
+<junction x="45.085" y="189.865"/>
+<pinref part="C2" gate="G$1" pin="2"/>
+<wire x1="55.245" y1="196.215" x2="55.245" y2="189.865" width="0.1524" layer="91"/>
+<junction x="55.245" y="189.865"/>
 </segment>
 <segment>
@@
 <net name="N$8" class="0">
 <segment>
+<wire x1="59.055" y1="229.235" x2="38.735" y2="229.235" width="0.1524" layer="91" grouprefs="POWER_SUPPLY EXTERNAL_USB_POWER_SUPPLY_INPUT"/>
+<pinref part="CN1" gate="G$1" pin="CC1"/>
 <pinref part="R3" gate="G$1" pin="1"/>
-<wire x1="59.055" y1="229.235" x2="38.735" y2="229.235" width="0.1524" layer="91" grouprefs="POWER_SUPPLY EXTERNAL_USB_POWER_SUPPLY_INPUT"/>
-<wire x1="38.735" y1="229.235" x2="38.735" y2="221.615" width="0.1524" layer="91" grouprefs="POWER_SUPPLY EXTERNAL_USB_POWER_SUPPLY_INPUT"/>
-<pinref part="CN1" gate="G$1" pin="CC1"/>
+<wire x1="38.735" y1="221.615" x2="38.735" y2="229.235" width="0.1524" layer="91"/>
 </segment>
 </net>
@@
 <net name="N$10" class="0">
 <segment>
-<pinref part="R4" gate="G$1" pin="1"/>
 <wire x1="59.055" y1="208.915" x2="55.245" y2="208.915" width="0.1524" layer="91" grouprefs="POWER_SUPPLY EXTERNAL_USB_POWER_SUPPLY_INPUT"/>
+<pinref part="CN1" gate="G$1" pin="SHIELD"/>
+<pinref part="R4" gate="G$1" pin="2"/>
 <wire x1="55.245" y1="208.915" x2="45.085" y2="208.915" width="0.1524" layer="91" grouprefs="POWER_SUPPLY EXTERNAL_USB_POWER_SUPPLY_INPUT"/>
-<wire x1="45.085" y1="208.915" x2="45.085" y2="205.105" width="0.1524" layer="91" grouprefs="POWER_SUPPLY EXTERNAL_USB_POWER_SUPPLY_INPUT"/>
-<pinref part="C2" gate="G$1" pin="2"/>
-<wire x1="55.245" y1="203.835" x2="55.245" y2="208.915" width="0.1524" layer="91" grouprefs="POWER_SUPPLY EXTERNAL_USB_POWER_SUPPLY_INPUT"/>
-<junction x="55.245" y="208.915" grouprefs="POWER_SUPPLY EXTERNAL_USB_POWER_SUPPLY_INPUT"/>
-<pinref part="CN1" gate="G$1" pin="SHIELD"/>
-</segment>
-</net>
+<wire x1="45.085" y1="205.105" x2="45.085" y2="208.915" width="0.1524" layer="91"/>
+<pinref part="C2" gate="G$1" pin="1"/>
+<wire x1="55.245" y1="203.835" x2="55.245" y2="208.915" width="0.1524" layer="91"/>
+<junction x="55.245" y="208.915"/>
+</segment>
+</net>

Commit message: Schematic v1.1 release
- Minor improvements on parts designators position;
- Just one resistor as pull up in not used pins at OLED display.
Parts:
- removed R26: 10k (5%), My-RLC:R_0603
- R10, R12: value 10k (1%) -> 10k (5%)
- R4: value 1M (1%) -> 1M (5%)
- R9: value 5k1 (1%) -> 5k1 (5%); SPICEPREFIX (none) -> R
Connections:
- removed net N$2: DS1.!D/C, R26.1
- net !DISPLAY_OLED_RESET: now also DS1.D/!C
- net 3.3V: no longer R26.2
- net N$3: now also DS1.E/!RD, DS1.R/!W; no longer DS1.!E/RD, DS1.!R/W
Other:
- note added: "Charge Pump for internal voltage regulator (only used when VBAT ≠ VDD)"
- note removed: "SA0"
- note removed: "SDA-SCL"
- moved on the sheet: C1, Q2, Q3, R1, R10, R11, R12, R2, R5, R8, U1

Commit message: Board design WIP
Parts:
- K1: device My-Relays:DPDT -> My-Relays:DPDT-SMD
Changed lines of the file:
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@@
 </part>
 <part name="SUPPLY19" library="My-Supply" library_urn="urn:adsk.eagle:library:35531236" deviceset="VBUS" device=""/>
-<part name="K1" library="My-Relays" library_urn="urn:adsk.eagle:library:35802173" deviceset="DPDT" device="" package3d_urn="urn:adsk.eagle:package:35802206/2"/>
+<part name="K1" library="My-Relays" library_urn="urn:adsk.eagle:library:35802173" deviceset="DPDT" device="-SMD" package3d_urn="urn:adsk.eagle:package:35848296/1" override_package3d_urn="urn:adsk.eagle:package:35848300/2" override_package_urn="urn:adsk.eagle:footprint:35848295/1"/>
 <part name="CN2" library="My-Connectors" library_urn="urn:adsk.eagle:library:35513533" deviceset="3P-" device="MINI-FIT-JR" package3d_urn="urn:adsk.eagle:package:35802278/2"/>
 <part name="SUPPLY23" library="My-Supply" library_urn="urn:adsk.eagle:library:35531236" deviceset="0V" device=""/>

Commit message: PCB v1.0 release
Parts:
- removed C21: 100nF, My-RLC:C_0603
- removed DS1: 0.96" active Area / 128x64 pixels, My-Displays:OLED-RAW-0.96"
- removed R20: 100R (5%), My-RLC:R_0603
- removed R21, R22: 4k7 (5%), My-RLC:R_0603
- removed R23: 390k (1%), My-RLC:R_0603
- removed R24, R25: 10k (5%), My-RLC:R_0603
- C1: value 100nF -> 4.7nF x 100V; PARTNO GRM155R71H104KE14D -> (none); PN C0603C104M5RACTU -> (none)
- C10: value 100nF -> 100nF x 50V; PARTNO GRM155R71H104KE14D -> (none); PN C0603C104M5RACTU -> (none)
- C11: value 1nF -> 100nF; PARTNO GRJ155R60J106ME11D -> *; PN GRM188R61A106ME69D -> (none)
- C12: value 100uF x 10V -> 100nF; device My-RLC:CP_5MM -> My-RLC:C_0603; PARTNO (none) -> *
- C13: PARTNO GRM155R71H104KE14D -> *; PN C0603C104M5RACTU -> (none)
- C14: PARTNO GRM155R71H104KE14D -> GRJ155R60J106ME11D; PN C0603C104M5RACTU -> GRM188R61A106ME69D
- C15: value 100nF -> 10nF; PARTNO * -> (none)
- C16: value 100nF -> 100uF x 10V; device My-RLC:C_0603 -> My-RLC:CP_5MM; PARTNO * -> (none)
- C17: value 10uF -> 10uF x 10V; device My-RLC:C_0603 -> My-RLC:CP_1206_POL; DESCRIPTION (none) -> Tantalum Electrolytic Capacitors (Low ESR); PARTNO GRM155R71H104KE14D -> (none); PN C0603C104M5RACTU -> (none)
- C18, C9: value 10uF -> 100nF x 50V; PARTNO GRJ155R60J106ME11D -> (none); PN GRM188R61A106ME69D -> (none)
- C19: value 10uF -> 22uF x 6.3V; device My-RLC:C_0603 -> My-RLC:CP_1206_POL; DESCRIPTION (none) -> Tantalum Electrolytic Capacitors (Low ESR); PARTNO GRM155R71H104KE14D -> (none); PN C0603C104M5RACTU -> (none); SPICEPREFIX C -> (none)
- C2: value 4.7nF -> 100nF x 50V; PARTNO GRM155R72A472KA01D -> (none)
- C20: value 1uF -> 100nF x 50V; PARTNO * -> (none)
- C3: value 100nF -> 10uF x 6.3V; PARTNO GRM155R71H104KE14D -> (none)
- C4: value 10uF -> 10uF x10V; PARTNO GRJ155R60J106ME11D -> (none)
- C5: value 100nF -> 1nF x 50V; PARTNO * -> (none)
- C6: value 10nF -> 10uF x 6.3V
- C7: value 10uF -> 1uF x 6.3V; PARTNO GRJ155R60J106ME11D -> (none); PN GRM188R61A106ME69D -> (none)
- C8: value 1nF -> 1nF x 50V; PARTNO GRJ155R60J106ME11D -> (none); PN GRM188R61A106ME69D -> (none)
- CN1: value USB 3.2 Gen 2 Type C Receptacle -> USB Type C Receptacle; device My-Connectors:USB-C -> My-Connectors:USB-C-16P-2LAYERS; PARTNO USB4080-03-A -> (none)
- CN2: value 3P-MINI-FIT-JR -> OLED-MODULE-I2C-SOCKET; device My-Connectors:3P-MINI-FIT-JR -> My-Displays:OLED-MODULE-I2C-SOCKET; FAMILY (none) -> SSD1306 (Display Driver and Controller)
- CN4: value JTAG -> CR1220; device My-Connectors:JTAG -> My-Battery:CELL-HARWIN; PARTNO FTSH-105-01-L-DV-K -> *
- CN5: value CELL-CONNECTOR -> BATTERY; device My-Battery:CELL-CONNECTOR -> My-Battery:CELL-JST-PH-2P-H; CAPACITY (none) -> 230mAh; TYPE (none) -> Li-Po; VOLTAGE (none) -> 3.7V~4.2V
- CN6: value CR-1220 -> 3P-MINI-FIT-JR; device My-Battery:CR-1220 -> My-Connectors:3P-MINI-FIT-JR; PARTNO * -> (none)
- Q1: value BC817 -> NPN-BC817; PN BC817K-16HR -> (none)
- Q2: PARTNO PMMT491A,215 -> (none)
- Q3: value NPN-BC817 -> BC817; PARTNO PMMT491A,215 -> (none); PN (none) -> BC817K-16HR
- R1: value 22R (5%) -> 1M (5%); PARTNO RC0402FR-1322RL -> (none); PN RC0603JR-0724KL -> (none)
- R10: value 10k (5%) -> 22K (5%); PARTNO RC0402FR-0710KL -> *; PN RC0603JR-0710KL -> (none)
- R11: value 4k7 (5%) -> 10k (5%); PARTNO RC0402JR-074K7L -> (none); PN RC0603JR-074K7L -> RC0603JR-0710KL
- R12: value 10k (5%) -> 47R (5%); PARTNO RC0402FR-0710KL -> (none); PN RC0603JR-0710KL -> (none)
- R13: value 47R (5%) -> 4k7 (5%); PN (none) -> RC0603JR-074K7L
- R14: value 22K (5%) -> 10k (5%); PARTNO * -> (none)
- R15: value 24k (5%) -> 100R (5%); PARTNO RC0402FR-0724KL -> (none); PN RC0603JR-0724KL -> (none)
- R16: value 47k (5%) -> 24k (5%); PARTNO RC0402FR-0747KL -> RC0402FR-0724KL; PN RC0603JR-1047KL -> RC0603JR-0724KL
- R17: value 10k (5%) -> 47k (5%); PARTNO (none) -> RC0402FR-0747KL; PN (none) -> RC0603JR-1047KL
- R2: value 22R (5%) -> 4k7 (5%); PARTNO RC0402FR-1322RL -> (none); PN RC0603JR-0724KL -> (none)
- R3: PARTNO AC0402FR-075K1L -> (none)
- R4: value 1M (5%) -> 5k1 (1%); PARTNO RC0402JR-071ML -> (none)
- R5: PARTNO RC0402FR-0722KL -> (none); PN RC0603JR-0722KL -> (none)
- R6: value 10k (5%) -> 4k7 (5%); PN RC0603JR-0710KL -> (none)
- R7: value 4k7 (5%) -> 10k (5%); PN RC0603JR-074K7L -> (none)
- R8: PARTNO RC0402JR-074K7L -> (none); PN RC0603JR-074K7L -> (none)
- R9: value 5k1 (5%) -> 4k7 (5%); PARTNO AC0402FR-075K1L -> (none); SPICEPREFIX R -> (none)
- SOC1: value ESP32-WROOM-32E-N4 -> ESP32-WROOM-32E; PARTNO ESP32-WROOM-32E(M113EH3200PH3Q0) -> (none)
- U1: PARTNO CP2102N-A02-GQFN28 -> (none); PN CP2102N-A02-GQFN28 -> (none)
- U2: value LMV321 -> MCP73831; device My-OpAmps:SINGLE -> My-ICs:MCP73831T-2ACI/OT; PARTNO (none) -> *
- U3: value MCP73831 -> LMV321; device My-ICs:MCP73831T-2ACI/OT -> My-OpAmps:SINGLE-LMV321; PARTNO * -> (none)
- U4: value TLV75530PDBVR -> DS3231-SO16; device My-LDOs:TLV75530PDBVR -> My-ICs:DS3231-SO16; PARTNO * -> (none)
- U5: value DS3231-SO16 -> 1117-3.3V; device My-ICs:DS3231-SO16 -> My-LDOs:1117-3.3V; FAMILY (none) -> NCP1117-3.3
Connections:
- net ESP32_UART_RX_USB renamed USB_TX
- net ESP32_UART_TX_USB renamed USB_RX
- removed net !DISPLAY_OLED_RESET: DS1.!RES, DS1.D/!C, R24.1
- removed net ESP32_ADC_BATTERY_SUPPLY_MONITOR: R18.1, R19.2, SOC1.IO36
- removed net ESP32_GPIO_PROG_ENABLE: C7.1, C8.1, CN4.!RST, Q2.C, R10.2, SOC1.EN
- removed net ESP32_GPIO_PROG_MODE: C11.1, Q3.C, R12.2, SOC1.IO0
- removed net ESP32_I2C_SCL: DS1.D0, R22.1, SOC1.IO22, U5.SCL
- removed net ESP32_I2C_SDA: DS1.D1, DS1.D2, R21.1, SOC1.IO21, U5.SDA
- removed net ESP32_USB_RTS: Q2.E, R11.1, U1.RTS
- removed net JTAG_TCK: CN4.TCK, SOC1.IO13
- removed net JTAG_TDI: CN4.TDI, SOC1.IO12
- removed net JTAG_TDO: CN4.TDO, SOC1.IO15
- removed net JTAG_TMS: CN4.TMS, SOC1.IO14
- removed net N$10: C2.1, CN1.SHIELD, R4.2
- removed net N$13: Q2.B, R8.1
- removed net N$16: Q3.B, R11.2
- removed net N$18: R5.2, U1.!RST
- removed net N$19: R1.2, U1.D-
- removed net N$20: Q3.E, R8.2, U1.DTR
- removed net N$21: CN1.CC2, R9.1
- removed net N$22: R2.2, U1.D+
- removed net USB_N: CN1.DN1, CN1.DN2, R1.1
- removed net USB_P: CN1.DP1, CN1.DP2, R2.1
- new net ESP32_ADC_BATTERY_SMONITOR: R18.1, R19.2, SOC1.IO35
- new net ESP32_PROG_ENABLE: C3.1, C5.1, Q1.C, R5.2, SOC1.EN
- new net ESP32_PROG_MODE: C8.1, Q2.C, R7.2, SOC1.IO0
- new net I2C_SCL: CN2.SCL, R9.1, SOC1.IO22, U4.SCL
- new net I2C_SDA: CN2.SDA, R8.1, SOC1.IO21, U4.SDA
- new net N$2: CN1.CC1, R4.1
- new net N$79: C1.2, CN1.S1, CN1.S2, CN1.S3, CN1.S4, R1.1
- new net USB_DTR: Q2.E, R2.2, U1.DTR
- new net USB_RTS: Q1.E, R6.2, U1.RTS
- net 0V: now also C1.1, C10.1, C12.1, C13.1, C15.2, C16.-, C17.-, C19.-, C2.1, C3.2, C5.2, C7.1, CN1.GND, CN2.GND, CN4.-, Q3.E, R1.2, R10.1, R11.2, R17.2, R4.2, U2.VSS, U3G$1.V-; no longer C1.2, C10.2, C12.-, C13.2, C15.1, C16.2, C17.2, C19.2, C2.2, C21.2, C3.1, C5.1, C7.2, CN1.GND_A, CN1.GND_B, CN4.GND, CN4.GND2, CN4.GND3, CN6.-, DS1.BS0, DS1.BS2, DS1.VLSS, DS1.VSS, Q1.E, R16.2, R17.1, R23.1, R25.1, R4.1, R6.2, R9.2, U2G$1.V-, U3.VSS
- net 3.3V: now also C10.2, C11.1, C12.2, C13.2, C19.+, C6.1, C7.2, CN2.VCC, R7.1, R8.2, R9.2, U3G$1.V+, U4.VDD, U5.OUT; no longer C1.1, C10.1, C13.1, C14.1, C15.2, C21.1, C5.2, CN4.VDD, DS1.BS1, DS1.VBAT, DS1.VDD, R10.1, R12.1, R21.2, R22.2, R24.2, U2G$1.V+, U4.OUT, U5.VDD
- net ESP32_ADC_TASK_FEEDBACK_MONITOR: now also C15.1, R12.2, SOC1.IO27; no longer C6.1, R13.2, SOC1.IO26
- net ESP32_GPIO_BATTERY_CHARGING_STATUS: now also SOC1.IO26, U2.STAT; no longer SOC1.IO34, U3.STAT
- net ESP32_GPIO_EXTERNAL_SUPPLY_MONITOR: now also R16.2, R17.1, SOC1.IO34; no longer R15.2, R16.1, SOC1.IO39, U1.VBUS
- net ESP32_GPIO_TASK_CONTROLLER: now also R11.1, R13.2, SOC1.IO25; no longer R6.1, R7.2, SOC1.IO32
- net N$1: now also CN1.CC2, R3.1; no longer C19.1, DS1.VCOMH
- net N$11: now also R15.2; no longer R20.2
- net N$12: now also R12.1, U3-A.-IN, U3-A.OUT; no longer R13.1, U2-A.-IN, U2-A.OUT
- net N$14: now also CN6-2.P$1; no longer CN2-2.P$1
- net N$15: now also CN6-3.P$1; no longer CN2-3.P$1
- net N$26: now also R10.2, U2.PROG; no longer R14.2, U3.PROG
- net N$3: now also CN1.D-, U1.D-; no longer DS1.!CS, DS1.D3, DS1.D4, DS1.D5, DS1.D6, DS1.D7, DS1.E/!RD, DS1.R/!W, R25.2
- net N$4: now also U3-A.+IN; no longer U2-A.+IN
- net N$41: now also Q3.B, R13.1; no longer Q1.B, R7.1
- net N$42: now also Q3.C; no longer Q1.C
- net N$5: now also CN6-1.P$1; no longer CN2-1.P$1
- net N$6: now also CN1.D+, U1.D+; no longer DS1.IREF, R23.2
- net N$7: now also Q1.B, R2.1; no longer C17.1, DS1.VCC
- net N$8: now also Q2.B, R6.1; no longer CN1.CC1, R3.1
- net P$1: now also U2.VBAT; no longer U3.VBAT
- net RTC_VBAT: now also C14.1, CN4.+, U4.VBAT; no longer C18.1, CN6.+, U5.VBAT
- net VBUS: now also C2.2, CN1.VBUS, R14.2, R16.1, U1.VBUS, U2.VDD; no longer C3.2, CN1.VBUS_A, CN1.VBUS_B, R17.2, R20.1, U3.VDD
- net VSYS: now also C16.+, C17.+, C18.1, U5.IN; no longer C12.+, C16.1, U4.EN, U4.IN
Other:
- note added: "* Built-in hall effect sensor: 29.4 chapter from Technical Reference Manual v4.6"
- note added: "* Only input: 3.2 chapter from datasheet v1.3"
- note added: "* Strapping pins: 3.3 chapter from datasheet v1.3"
- note added: "I2C"
- note added: "Serial Bootloader Programmer Interface"
- note added: "USB Self-Powered mode with internal 3.3V LDO bypassed"
- note removed: "!JTAG/RST"
- note removed: "* Only used when communicating protocol = 8-bit parallel mode"
- note removed: "* Only used when communicating protocol = SPI mode"
- note removed: "238mV drops at 500mA"
- note removed: "7-bits Slave Address 0b0111101 0x3D"
- note removed: "= I2C mode"
- note removed: "Built-in hall effect sensor: 29.4 chapter from Technical Reference Manual v4.6"
- note removed: "Charge Pump for internal voltage regulator (only used when VBAT ≠ VDD)"
- note removed: "Communicating Protocol Select"
- note removed: "IQ = 25μA"
- note removed: "In-Circuit Programmer and Debugger Interface"
- note removed: "Only input: 3.2 chapter from datasheet v1.3"
- note removed: "SDA"
- note removed: "SDA-IN"
- note removed: "SDA-OUT"
- note removed: "Strapping pins: 3.3 chapter from datasheet v1.3"
- moved on the sheet: C1, C10, C11, C13, C14, C15, C18, C2, C20, C3, C4, C5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
